File: board_stm32/board_stm32.sch (EAGLE design)
At the start: 8 parts, among them IC2 NE555, T1 BC547

Commit message: update schematic and board, add .gitignore
Parts:
- removed B1: ARDUINO_MEGA_R3FULL, SparkFun-Boards:ARDUINO_MEGA_R3FULL
- removed C1: (no value), rcl:CPOL-USE2.5-6
- removed IC2: NE555, st-microelectronics:NE555
- removed R1, R2, R3: (no value), rcl:R-EU_0204/7
- removed S1: MOMENTARY-SWITCH-SPST-PTH-6.0MM, SparkFun-Switches:MOMENTARY-SWITCH-SPST-PTH-6.0MM
- removed T1: BC547, transistor:BC547
- added JP1: (no value), adafruit:PINHD-1X6
- added U$1: STM32F411CEU6, STM32F411CEU6:STM32F411CEU6
Connections:
- removed net 5V: B1.5V, IC2./RES, IC2.VCC+, R2.2, R3.2
- removed net N$1: C1.+, IC2.DIS, IC2.TRE, R3.1
- removed net N$2: IC2.OUT, R1.1
- removed net N$3: R1.2, T1.B
- removed net RST: B1.!RESET, R2.1, S1.2, T1.C
- removed net RST_GPIO: B1.7, IC2.TRI
- new net CS: JP1.6, U$1.B12
- new net MISO: JP1.3, U$1.B14
- new net MOSI: JP1.4, U$1.B15
- new net SCK: JP1.5, U$1.B13
- new net VCC: JP1.2, U$1.5V, U$1.5V_2
- net GND: now also JP1.1, U$1.GND, U$1.GND_2; no longer B1.GND, B1.GND@2, C1.-, IC2.GND, S1.1, T1.E

Commit message: redesign PCB
Parts:
- added JP2, JP3: (no value), adafruit:PINHD-1X1
Connections:
- new net N$1: JP2.1, U$1.R
- net GND: now also JP3.1
Changed lines of the file:
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@@
 <part name="U$1" library="STM32F411CEU6" deviceset="STM32F411CEU6" device=""/>
 <part name="JP1" library="adafruit" deviceset="PINHD-1X6" device=""/>
+<part name="JP2" library="adafruit" deviceset="PINHD-1X1" device=""/>
+<part name="JP3" library="adafruit" deviceset="PINHD-1X1" device=""/>
 </parts>
 <sheets>
@@
 <attribute name="NAME" x="65.405" y="52.07" size="1.778" layer="95" rot="R90"/>
 <attribute name="VALUE" x="86.36" y="52.07" size="1.778" layer="96" rot="R90"/>
+</instance>
+<instance part="JP2" gate="G$1" x="0" y="50.8" smashed="yes" rot="R90">
+<attribute name="NAME" x="-3.175" y="44.45" size="1.778" layer="95" rot="R90"/>
+<attribute name="VALUE" x="5.08" y="44.45" size="1.778" layer="96" rot="R90"/>
+</instance>
+<instance part="JP3" gate="G$1" x="-17.78" y="50.8" smashed="yes" rot="R90">
+<attribute name="NAME" x="-20.955" y="44.45" size="1.778" layer="95" rot="R90"/>
+<attribute name="VALUE" x="-12.7" y="44.45" size="1.778" layer="96" rot="R90"/>
 </instance>
 </instances>
@@
 <wire x1="12.7" y1="12.7" x2="5.08" y2="12.7" width="0.1524" layer="91"/>
 <label x="5.08" y="12.7" size="1.778" layer="95" rot="R180"/>
+</segment>
+<segment>
+<pinref part="JP3" gate="G$1" pin="1"/>
+<wire x1="-17.78" y1="48.26" x2="-17.78" y2="40.64" width="0.1524" layer="91"/>
+<label x="-17.78" y="40.64" size="1.778" layer="95" rot="R180"/>
 </segment>
 </net>
@@
 </segment>
 </net>
+<net name="N$1" class="0">
+<segment>
+<pinref part="JP2" gate="G$1" pin="1"/>
+<pinref part="U$1" gate="G$1" pin="R"/>
+<wire x1="0" y1="48.26" x2="12.7" y2="48.26" width="0.1524" layer="91"/>
+</segment>
+</net>
